File: MCP3909_Breakout/MCP3909_Breakout.kicad_pcb (KiCad board)
At the start: 2 copper layers, 1 part

Commit message: First go at place-n-route
Parts:
- added C1: 33n, Capacitor_SMD:C_0603_1608Metric, F.Cu at (152.1, 105.4)
- added C10: 15p, Capacitor_SMD:C_0603_1608Metric, F.Cu at (134.6, 89.7)
- added C11: 4.7u, Capacitor_SMD:C_0805_2012Metric, F.Cu at (134.1, 101.6)
- added C12: 100n, Capacitor_SMD:C_0603_1608Metric, F.Cu at (136.7, 101.3)
- added C2: 33n, Capacitor_SMD:C_0603_1608Metric, F.Cu at (150.4, 105.4)
- added C3: 33n, Capacitor_SMD:C_0603_1608Metric, F.Cu at (143.6, 105.9)
- added C4: 33n, Capacitor_SMD:C_0603_1608Metric, F.Cu at (140.3, 105.9)
- added C5: 100p, Capacitor_SMD:C_0603_1608Metric, F.Cu at (151.1, 102.6)
- added C6: 100n, Capacitor_SMD:C_0603_1608Metric, F.Cu at (148.6, 97.5)
- added C7: 100n, Capacitor_SMD:C_0603_1608Metric, F.Cu at (136.7, 94.7)
- added C8: 4.7u, Capacitor_SMD:C_0805_2012Metric, F.Cu at (134.1, 94.5)
- added C9: 15p, Capacitor_SMD:C_0603_1608Metric, F.Cu at (151.9, 89.7)
- added FB1: FerriteBead_Small, Inductor_SMD:L_0603_1608Metric, F.Cu at (134.1, 98.0)
- added FB2: FerriteBead_Small, Inductor_SMD:L_0603_1608Metric, F.Cu at (131.6, 98.0)
- added J1: Conn_01x10, Connector_PinHeader_2.54mm:PinHeader_1x10_P2.54mm_Vertical, F.Cu at (132.1, 112.0)
- added JP1: SolderJumper_3_Bridged12, Jumper:SolderJumper-3_P1.3mm_Bridged12_RoundedPad1.0x1.5mm, B.Cu at (132.3, 94.0)
- added JP2: SolderJumper_3_Bridged12, Jumper:SolderJumper-3_P1.3mm_Bridged12_RoundedPad1.0x1.5mm, B.Cu at (132.3, 99.6)
- added R1: 2R2, Resistor_SMD:R_0603_1608Metric, F.Cu at (149.4, 108.5)
- added R2: 2R2, Resistor_SMD:R_0603_1608Metric, F.Cu at (153.2, 108.5)
- added R3: 1k, Resistor_SMD:R_0603_1608Metric, F.Cu at (143.6, 107.7)
- added R4: 1k, Resistor_SMD:R_0603_1608Metric, F.Cu at (140.3, 107.7)
- added R5: 1k, Resistor_SMD:R_0603_1608Metric, F.Cu at (153.9, 105.4)
- added R6: 1k, Resistor_SMD:R_0603_1608Metric, F.Cu at (148.6, 105.4)
- added TP1: TestPoint, TestPoint:TestPoint_Pad_1.5x1.5mm, B.Cu at (128.1, 94.0)
- added TP2: TestPoint, TestPoint:TestPoint_Pad_1.5x1.5mm, B.Cu at (128.1, 97.5)
- added TP3: TestPoint, TestPoint:TestPoint_Pad_1.5x1.5mm, B.Cu at (128.1, 101.1)
- added TP4: TestPoint, TestPoint:TestPoint_Pad_1.5x1.5mm, B.Cu at (128.1, 104.6)
- added Y1: Crystal_Small, Crystal:Crystal_SMD_HC49-SD, F.Cu at (143.3, 89.4)
- moved U1 2.62 mm to (143.0, 97.8), turned to 90 degrees
Connections:
- U1 pad 1: unconnected-(U1-DVDD-Pad1) -> VIN
- U1 pad 10: unconnected-(U1-REFIN/OUT-Pad10) -> Net-(U1-REFIN/OUT)
- U1 pad 11: unconnected-(U1-AGND-Pad11) -> GND
- U1 pad 12: unconnected-(U1-SCK/F2-Pad12) -> SCK/F2
- U1 pad 13: unconnected-(U1-SDI/F1-Pad13) -> MOSI/F1
- U1 pad 14: unconnected-(U1-~{CS}/F0-Pad14) -> ~{CS}/F0
- U1 pad 15: unconnected-(U1-G1-Pad15) -> G1
- U1 pad 16: unconnected-(U1-G0-Pad16) -> G0
- U1 pad 17: unconnected-(U1-OSC1-Pad17) -> Net-(U1-OSC1)
- U1 pad 18: unconnected-(U1-OSC2-Pad18) -> Net-(U1-OSC2)
- U1 pad 2: unconnected-(U1-HPF-Pad2) -> VIN
- U1 pad 20: unconnected-(U1-SDO/NEG-Pad20) -> MISO/NEG
- U1 pad 21: unconnected-(U1-DGND-Pad21) -> GNDD
- U1 pad 22: unconnected-(U1-HFOUT-Pad22) -> HFOUT
- U1 pad 23: unconnected-(U1-FOUT1-Pad23) -> FOUT1
- U1 pad 24: unconnected-(U1-FOUT0-Pad24) -> FOUT0
- U1 pad 3: unconnected-(U1-AVDD-Pad3) -> Net-(U1-AVDD)
- U1 pad 5: unconnected-(U1-CH0+-Pad5) -> IAP
- U1 pad 6: unconnected-(U1-CH0--Pad6) -> IAN
- U1 pad 7: unconnected-(U1-CH1--Pad7) -> UN
- U1 pad 8: unconnected-(U1-CH1+-Pad8) -> UP
- U1 pad 9: unconnected-(U1-~{MCLR}-Pad9) -> ~{MCLR}
Routing:
- net GND: track 0.00 -> 90.8 mm, vias 0 -> 1
- net SCK/F2: track 0.00 -> 66.6 mm, vias 0 -> 2
- net ~{MCLR}: track 0.00 -> 38.6 mm, vias 0 -> 1
- net VIN: track 0.00 -> 35.0 mm, vias 0 -> 2
- net ~{CS}/F0: track 0.00 -> 26.2 mm, vias 0 -> 1
- net HFOUT: track 0.00 -> 22.2 mm, vias 0 -> 1
- net FOUT1: track 0.00 -> 22.1 mm, vias 0 -> 1
- net MISO/NEG: track 0.00 -> 22.0 mm, vias 0 -> 1
- net MOSI/F1: track 0.00 -> 21.7 mm, vias 0 -> 1
- net UP: track 0.00 -> 17.8 mm, vias 0 -> 2
- net G1: track 0.00 -> 16.0 mm, vias 0 -> 1
- net IAN: track 0.00 -> 15.4 mm
- net UN: track 0.00 -> 15.3 mm, vias 0 -> 2
- net G0: track 0.00 -> 14.7 mm, vias 0 -> 1
- net GNDD: track 0.00 -> 14.4 mm
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- added copper zone on B.Cu, net GND
- added copper zone on F.Cu, net GND
Other:
- board outline added: 38.1 x 27.9 mm

Commit message: Complete routing
Parts:
- added SYM1: Logo_Open_Hardware_Small, Symbol:OSHW-Logo2_9.8x8mm_SilkScreen, B.Cu at (144.8, 100.3)
Other:
- board text added: "FOUT0"
- board text added: "FOUT1"
- board text added: "G0"
- board text added: "G1"
- board text added: "GND"
- board text added: "HFOUT"
- board text added: "IAN"
- board text added: "IAP"
- board text added: "MAX Vrms = 470mV - Ch0 MAX Vrms = 660mV - Ch1 MCP3909 Breakout"
- board text added: "MISO"
- board text added: "MOSI"
- board text added: "SCK"
- board text added: "UN"
- board text added: "UP"
- board text added: "VIN"
- board text added: "by Tisham Dhar https://whatnick.com v0.1 29/03/2025"
- board text added: "~{CS}"
- board text added: "~{MCLR}"

Commit message: Produce fabrication outputs
Parts:
- U1: value ~ -> MCP3909
Changed lines of the file:
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@@
       (outputformat 1)
       (mirror false)
-      (drillshape 1)
+      (drillshape 0)
       (scaleselection 1)
-      (outputdirectory "")
+      (outputdirectory "gerbers")
     )
   )
@@
     (descr "Inductor SMD 0603 (1608 Metric), square (rectangular) end terminal, IPC_7351 nominal, (Body size source: http://www.tortai-tech.com/upload/download/2011102023233369053.pdf), generated with kicad-footprint-generator")
     (tags "inductor")
+    (property "MPN" "BLM03AG100SN1D")
     (property "Sheetfile" "MCP3909_Breakout.kicad_sch")
     (property "Sheetname" "")
@@
     (descr "Inductor SMD 0603 (1608 Metric), square (rectangular) end terminal, IPC_7351 nominal, (Body size source: http://www.tortai-tech.com/upload/download/2011102023233369053.pdf), generated with kicad-footprint-generator")
     (tags "inductor")
+    (property "MPN" "BLM03AG100SN1D")
     (property "Sheetfile" "MCP3909_Breakout.kicad_sch")
     (property "Sheetname" "")
@@
     (descr "24-Lead Plastic Shrink Small Outline (SS)-5.30 mm Body [SSOP] (see Microchip Packaging Specification 00000049BS.pdf)")
     (tags "SSOP 0.65")
+    (property "MPN" "MCP3909")
     (property "Sheetfile" "MCP3909_Breakout.kicad_sch")
     (property "Sheetname" "")
@@
         (effects (font (size 0.8 0.8) (thickness 0.2)))
     )
-    (fp_text value "~" (at 0 5.25 90) (layer "F.Fab")
-        (effects (font (size 1 1) (thickness 0.15)))
-    )
+    (fp_text value "MCP3909" (at 0 5.25 90) (layer "F.Fab")
+        (effects (font (size 1 1) (thickness 0.15)))
+    )
